File: niftykeyzjackboardredux.kicad_sch (KiCad schematic)
At the start: 6 parts

Commit message: update board
Connections:
- net at JP18.3 (Pin_3), JP20.T: no longer JP20.TN
- net at JP18.4 (Pin_4), JP19.T: no longer JP19.TN
- no-connect marks 1 -> 3
Changed lines of the file:
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@@
 (kicad_sch (version 20211123) (generator eeschema)
   (paper "A4")
-  (junction (at 109.22 45.085) (diameter 0) (color 0 0 0 0)
-  )
   (junction (at 40.64 47.625) (diameter 0) (color 0 0 0 0)
   )
@@
   (junction (at 40.64 57.785) (diameter 0) (color 0 0 0 0)
   )
-  (junction (at 81.915 44.45) (diameter 0) (color 0 0 0 0)
-  )
   (junction (at 40.64 55.245) (diameter 0) (color 0 0 0 0)
   )
+  (no_connect (at 109.22 43.18))
+  (no_connect (at 81.915 43.18))
   (no_connect (at 140.335 42.545))
-  (wire (pts (xy 37.465 52.705) (xy 109.22 52.705))
+  (wire (pts (xy 37.465 52.705) (xy 111.76 52.705))
     (stroke (width 0) (type default) (color 0 0 0 0))
   )
-  (wire (pts (xy 81.915 50.165) (xy 37.465 50.165))
-    (stroke (width 0) (type default) (color 0 0 0 0))
-  )
-  (wire (pts (xy 109.22 52.705) (xy 109.22 45.085))
-    (stroke (width 0) (type default) (color 0 0 0 0))
-  )
-  (wire (pts (xy 81.915 44.45) (xy 84.455 44.45))
-    (stroke (width 0) (type default) (color 0 0 0 0))
-  )
-  (wire (pts (xy 109.22 43.18) (xy 109.22 45.085))
+  (wire (pts (xy 37.465 50.165) (xy 84.455 50.165))
     (stroke (width 0) (type default) (color 0 0 0 0))
   )
@@
     (stroke (width 0) (type default) (color 0 0 0 0))
   )
-  (wire (pts (xy 81.915 43.18) (xy 81.915 44.45))
-    (stroke (width 0) (type default) (color 0 0 0 0))
-  )
   (wire (pts (xy 142.875 60.325) (xy 37.465 60.325))
     (stroke (width 0) (type default) (color 0 0 0 0))
@@
   )
   (wire (pts (xy 86.995 43.18) (xy 86.995 45.72))
-    (stroke (width 0) (type default) (color 0 0 0 0))
-  )
-  (wire (pts (xy 109.22 45.085) (xy 111.76 45.085))
     (stroke (width 0) (type default) (color 0 0 0 0))
   )
@@
     (stroke (width 0) (type default) (color 0 0 0 0))
   )
-  (wire (pts (xy 111.76 43.18) (xy 111.76 45.085))
+  (wire (pts (xy 111.76 43.18) (xy 111.76 52.705))
     (stroke (width 0) (type default) (color 0 0 0 0))
   )
@@
     (stroke (width 0) (type default) (color 0 0 0 0))
   )
-  (wire (pts (xy 81.915 44.45) (xy 81.915 50.165))
-    (stroke (width 0) (type default) (color 0 0 0 0))
-  )
   (wire (pts (xy 40.64 47.625) (xy 40.64 55.245))
     (stroke (width 0) (type default) (color 0 0 0 0))
@@
     (stroke (width 0) (type default) (color 0 0 0 0))
   )
-  (wire (pts (xy 84.455 44.45) (xy 84.455 43.18))
+  (wire (pts (xy 84.455 43.18) (xy 84.455 50.165))
     (stroke (width 0) (type default) (color 0 0 0 0))
   )
